File: Motor_Controller_Board/Motor_Board V5/_autosave-stepperDrivers.kicad_sch (KiCad schematic)
At the start: 60 parts, among them J401 Conn_01x04, J402 Conn_01x04, J403 Conn_01x04, U401 A4988, U402 A4988, U403 A4988

Commit message: done. see readme for update log
Parts:
- R401, R407, R412: value 24k -> 15k; LCSC Part Number C23352 -> C22809; MPN 0603WAF2402T5E -> 0603WAF1502T5E
- R404, R405, R413, R414, R420, R421: value 75m -> 100m; LCSC Part Number C149663 -> C188071; MPN CR1206FR075P05R -> RL12FTNR100; Manufacturer Ever Ohms Tech -> TA-I Tech
Other:
- note added: "I_trip = 2V / (8*0.075) = 2.5A"
- note added: "Vref <= 2V"
- note removed: "I_trip = .35 / (8*0.075) = 0.64A"
- note removed: "I_trip = 0.25 / (8*0.075) = 2A"
- note removed: "I_trip = 1.47 / (8*0.075) = 2.45A"
- note removed: "Vref = 0.25V"
- note removed: "Vref = 0.386V"
- note removed: "Vref = 1.47V"
