File: Motor_Controller_Board/Motor_Board V5/stepperDrivers.kicad_sch (KiCad schematic)
At the start: 60 parts, among them J401 Conn_01x04, J402 Conn_01x04, J403 Conn_01x04, U401 A4988, U402 A4988, U403 A4988

Commit message: cleaned up board and switched to horizontal text
Connections:
- net AGITATE_1A: now also U401.24 (OUT1A); no longer U401.21 (OUT1B)
- net AGITATE_1B: now also U401.21 (OUT1B); no longer U401.24 (OUT1A)
- net HORIZONTAL_1A: now also U402.24 (OUT1A); no longer U402.21 (OUT1B)
- net HORIZONTAL_1B: now also U402.21 (OUT1B); no longer U402.24 (OUT1A)
- net VERTICAL_1A: now also U403.24 (OUT1A); no longer U403.21 (OUT1B)
- net VERTICAL_1B: now also U403.21 (OUT1B); no longer U403.24 (OUT1A)
Changed lines of the file:
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@@
-	)
-	(junction
-		(at 72.39 135.89)
-		(diameter 0)
-		(color 0 0 0 0)
 	)
 	(junction
@@
 	(junction
 		(at 127 21.59)
-		(diameter 0)
-		(color 0 0 0 0)
-	)
-	(junction
-		(at 72.39 138.43)
 		(diameter 0)
 		(color 0 0 0 0)
@@
 	(wire
 		(pts
-			(xy 72.39 135.89) (xy 72.39 138.43)
-		)
-		(stroke
-			(width 0)
-			(type default)
-		)
-	)
-	(wire
-		(pts
 			(xy 73.66 146.05) (xy 73.66 148.59)
 		)
@@
 	(wire
 		(pts
-			(xy 71.12 138.43) (xy 72.39 138.43)
+			(xy 71.12 138.43) (xy 73.66 138.43)
 		)
 		(stroke
@@
 	(wire
 		(pts
-			(xy 72.39 138.43) (xy 73.66 138.43)
-		)
-		(stroke
-			(width 0)
-			(type default)
-		)
-	)
-	(wire
-		(pts
 			(xy 93.98 147.32) (xy 93.98 148.59)
 		)
@@
 	(wire
 		(pts
-			(xy 72.39 135.89) (xy 71.12 135.89)
+			(xy 71.12 135.89) (xy 76.2 135.89)
 		)
 		(stroke
@@
 		)
 		(stroke
-			(width 0)
-			(type default)
-		)
-	)
-	(wire
-		(pts
-			(xy 72.39 135.89) (xy 76.2 135.89)
-		)
-		(stroke

Commit message: done. see readme for update log
Parts:
- R401, R407, R412: value 24k -> 15k; LCSC Part Number C23352 -> C22809; MPN 0603WAF2402T5E -> 0603WAF1502T5E
- R404, R405, R413, R414, R420, R421: value 75m -> 100m; LCSC Part Number C149663 -> C188071; MPN CR1206FR075P05R -> RL12FTNR100; Manufacturer Ever Ohms Tech -> TA-I Tech
Other:
- note added: "I_trip = 2V / (8*0.075) = 2.5A"
- note added: "Vref <= 2V"
- note removed: "I_trip = .35 / (8*0.075) = 0.64A"
- note removed: "I_trip = 0.25 / (8*0.075) = 2A"
- note removed: "I_trip = 1.47 / (8*0.075) = 2.45A"
- note removed: "Vref = 0.25V"
- note removed: "Vref = 0.386V"
- note removed: "Vref = 1.47V"
